Commit message: update of values for sfnpod

File: hexapod_description/urdf/sfnpod_model.xacro (robot description, xacro)
@@ -3,9 +3,9 @@
 	<!-- parameters -->
 	<xacro:property name="pi" value="3.1415926535897931" />
-	<xacro:property name="body_length_x" value="0.250" />
-	<xacro:property name="body_length_y" value="0.125" />
-	<xacro:property name="coxa_length" value="0.052" />
-	<xacro:property name="femur_length" value="0.065" />
-	<xacro:property name="tibia_length" value="0.133" />
+	<xacro:property name="body_length_x" value="0.40" />
+	<xacro:property name="body_length_y" value="0.33" />
+	<xacro:property name="coxa_length" value="0.055" />
+	<xacro:property name="femur_length" value="0.140" />
+	<xacro:property name="tibia_length" value="0.220" />
     <gazebo>
         <plugin name="gazebo_ros_control" filename="libgazebo_ros_control.so">
@@ -19,15 +19,15 @@
         <origin xyz="0.0 0.0 0.0" rpy="0.0 0.0 0.0" />
     </joint>
-	<link name="body_link">
-			<visual>
-	  			<origin	xyz="0.0 0.0 0.0" rpy="0.0 0.0 0.0" />
-      			<geometry>
-        			<mesh filename="package://hexapod_description/meshes/phantomX/body.stl" scale="0.001 0.001 0.001"/>
-      			</geometry>
-				<material name="">
-					<color rgba="0.7 0.7 0.7 1" />
-				</material>
-			</visual>
-			<collision>
+    <link name="body_link">
+        <visual>
+            <origin xyz="0.0 0.0 0.0" rpy="0.0 0.0 0.0" />
+      	    <geometry>
+        	<mesh filename="package://hexapod_description/meshes/phantomX/body.stl" scale="0.001 0.001 0.001"/>
+      	    </geometry>
+	    <material name="">
+	         <color rgba="0.7 0.7 0.7 1" />
+	    </material>
+	</visual>
+        <collision>
             <origin xyz="0.0 0.0 0.0" rpy="0.0 0.0 0.0"/>
             <geometry>
@@ -50,6 +50,6 @@
         <material>Gazebo/DarkGrey</material>
     </gazebo>
-	<!-- Head Pan and Tilt properties -->
-	<joint name="head_pan_joint" type="revolute">
+    <!-- Head Pan and Tilt properties -->
+    <!--<joint name="head_pan_joint" type="revolute">
 		<parent link="body_link"/>
 		<child link="head_pan_link"/>
@@ -57,6 +57,6 @@
 		<origin xyz="0.145 0.0 0.080" />
 		<limit lower="-${3.14}" upper="${3.14}" effort="10000" velocity="100" />
-	</joint>
-	<link name="head_pan_link">
+    </joint>
+    <link name="head_pan_link">
         <inertial>
             <origin xyz="0.0 0.0 0.0" rpy="0.0 0.0 0.0" />
@@ -68,5 +68,5 @@
         </inertial>
     </link>
-	<joint name="head_tilt_joint" type="revolute">
+    <joint name="head_tilt_joint" type="revolute">
 		<parent link="head_pan_link"/>
 		<child link="head_tilt_link"/>
@@ -74,15 +74,15 @@
 		<origin xyz="0.0 0.0 0.020" />
 		<limit lower="-${3.14}" upper="${3.14}" effort="10000" velocity="100" />
-	</joint>
-	<link name="head_tilt_link">
-        <inertial>
-            <origin xyz="0.0 0.0 0.0" rpy="0.0 0.0 0.0" />
-            <mass value="0.00001"/>
-            <inertia
-                ixx="1.0" ixy="0.0"  ixz="0.0"
-                iyy="1.0" iyz="0.0"
-                izz="1.0" />
-        </inertial>
-    </link>
+    </joint>
+    <link name="head_tilt_link">
+        <inertial>
+            <origin xyz="0.0 0.0 0.0" rpy="0.0 0.0 0.0" />
+            <mass value="0.00001"/>
+            <inertia
+                ixx="1.0" ixy="0.0"  ixz="0.0"
+                iyy="1.0" iyz="0.0"
+                izz="1.0" />
+        </inertial>
+    </link>-->
 	<!-- IMU properties -->
 	<joint name="imu_joint" type="fixed">
@@ -105,5 +105,5 @@
 	<xacro:property name="joint_upper_limit" value="${3.14}" />
 	<xacro:property name="joint_effort" value="6.0" />
-	<xacro:property name="joint_velocity" value="0.524" />
+	<xacro:property name="joint_velocity" value="0.024" />
 	<!-- Leg macro -->
 	<xacro:macro name="leg" params="side position x y angle axis">

Commit message: changed some stuff, added a white box for the head and added a sitting height.

File: hexapod_description/urdf/sfnpod_model.xacro (robot description, xacro)
@@ -1,11 +1,11 @@
 <?xml version="1.0" encoding="UTF-8" ?>
 <robot xmlns:xacro="http://ros.org/wiki/xacro" name="sfnpod">
-	<!-- parameters -->
-	<xacro:property name="pi" value="3.1415926535897931" />
-	<xacro:property name="body_length_x" value="0.40" />
-	<xacro:property name="body_length_y" value="0.33" />
-	<xacro:property name="coxa_length" value="0.055" />
-	<xacro:property name="femur_length" value="0.140" />
-	<xacro:property name="tibia_length" value="0.220" />
+    <!-- parameters -->
+    <xacro:property name="pi" value="3.1415926535897931" />
+    <xacro:property name="body_length_x" value="0.40" />
+    <xacro:property name="body_length_y" value="0.33" />
+    <xacro:property name="coxa_length" value="0.055" />
+    <xacro:property name="femur_length" value="0.140" />
+    <xacro:property name="tibia_length" value="0.220" />
     <gazebo>
         <plugin name="gazebo_ros_control" filename="libgazebo_ros_control.so">
@@ -51,10 +51,10 @@
     </gazebo>
     <!-- Head Pan and Tilt properties -->
-    <!--<joint name="head_pan_joint" type="revolute">
-		<parent link="body_link"/>
-		<child link="head_pan_link"/>
-		<axis xyz="0.0 0.0 1.0" />
-		<origin xyz="0.145 0.0 0.080" />
-		<limit lower="-${3.14}" upper="${3.14}" effort="10000" velocity="100" />
+    <joint name="pan_joint" type="revolute">
+        <parent link="body_link"/>
+        <child link="head_pan_link"/>
+        <axis xyz="0.0 0.0 1.0" />
+        <origin xyz="0.145 0.0 0.080" />
+        <limit lower="-${3.14}" upper="${3.14}" effort="10000" velocity="100" />
     </joint>
     <link name="head_pan_link">
@@ -68,5 +68,5 @@
         </inertial>
     </link>
-    <joint name="head_tilt_joint" type="revolute">
+    <joint name="tilt_joint" type="revolute">
 		<parent link="head_pan_link"/>
 		<child link="head_tilt_link"/>
@@ -84,12 +84,37 @@
                 izz="1.0" />
         </inertial>
-    </link>-->
-	<!-- IMU properties -->
-	<joint name="imu_joint" type="fixed">
-		<parent link="base_link" />
-		<child link="imu_link" />
-		<origin xyz="0.0 0.0 0.0" rpy="0.0 0.0 0.0" />
-	</joint>
-	<link name="imu_link">
+    </link>
+    <!-- Joint to connect the head geometry to head_tilt_link -->
+    <joint name="head_geometry_joint" type="fixed">
+        <parent link="head_tilt_link"/>
+        <child link="head_geometry"/>
+        <origin xyz="0 0 0.02" rpy="0 0 0"/> <!-- Adjust position as needed -->
+    </joint>
+    <!-- Head geometry link definition -->
+    <link name="head_geometry">
+        <visual>
+            <geometry>
+                <box size="0.1 0.1 0.1"/> <!-- Adjust size as needed -->
+            </geometry>
+            <material name="head_color">
+                <color rgba="1 1 1 1"/> <!-- Set color as needed -->
+            </material>
+        </visual>
+        <inertial>
+            <origin xyz="0 0 0" rpy="0 0 0"/>
+            <mass value="0.1"/> <!-- Set mass as needed -->
+            <inertia
+                ixx="0.001" ixy="0" ixz="0"
+                iyy="0.001" iyz="0"
+                izz="0.001"/> <!-- Set inertia as needed -->
+        </inertial>
+    </link>
+    <!-- IMU properties -->
+    <joint name="imu_joint" type="fixed">
+        <parent link="base_link" />
+        <child link="imu_link" />
+        <origin xyz="0.0 0.0 0.0" rpy="0.0 0.0 0.0" />
+    </joint>
+    <link name="imu_link">
         <inertial>
             <origin xyz="0.0 0.0 0.0" rpy="0.0 0.0 0.0" />

Commit message: updated the sfn pod model with initial values for all joints.

File: hexapod_description/urdf/sfnpod_model.xacro (robot description, xacro)
@@ -132,5 +132,5 @@
 	<xacro:property name="joint_velocity" value="0.024" />
 	<!-- Leg macro -->
-	<xacro:macro name="leg" params="side position x y angle axis">
+	<xacro:macro name="leg" params="side position x y angle axis coxa_init femur_init tibia_init">
 		<!-- leg position -->
 		<joint name="leg_center_joint_${side}${position}" type="fixed">
@@ -156,4 +156,5 @@
 			<axis xyz="0.0 0.0 1.0" />
 			<limit lower="${joint_lower_limit}" upper="${joint_upper_limit}" effort="${joint_effort}" velocity="${joint_velocity}" />
+            <initial_position value="${coxa_init}"/>
 		</joint>
 		<transmission name="coxa_transmission_${side}${position}">
@@ -205,4 +206,5 @@
 			<axis xyz="0.0 0.0 ${-axis}" />
 			<limit lower="${joint_lower_limit}" upper="${joint_upper_limit}" effort="${joint_effort}" velocity="${joint_velocity}" />
+            <initial_position value="${femur_init}"/>
 		</joint>
 		<transmission name="femur_transmission_${side}${position}">
@@ -254,4 +256,5 @@
 			<axis xyz="0.0 0.0 ${axis}" />
 			<limit lower="${joint_lower_limit}" upper="${joint_upper_limit}" effort="${joint_effort}" velocity="${joint_velocity}" />
+            <initial_position value="${tibia_init}"/>
 		</joint>
 		<transmission name="tibia_transmission_${side}${position}">
@@ -298,9 +301,9 @@
 	</xacro:macro>
 	<!-- Build robot model -->
-	<xacro:leg side="R" position="R" x="-0.120" y="-0.060" angle="-${pi*3/4}" axis="1" />
-	<xacro:leg side="R" position="M" x="0.0" y="-0.100" angle="-${pi/2}" axis="1" />
-	<xacro:leg side="R" position="F" x="0.120" y="-0.060" angle="-${pi/4}" axis="1" />
-	<xacro:leg side="L" position="R" x="-0.120" y="0.060" angle="${pi*3/4}" axis="-1" />
-	<xacro:leg side="L" position="M" x="0.0" y="0.100" angle="${pi/2}" axis="-1" />
-	<xacro:leg side="L" position="F" x="0.120" y="0.060" angle="${pi/4}" axis="-1" />
+	<xacro:leg side="R" position="R" x="-0.120" y="-0.060" angle="-${pi*3/4}" axis="1" coxa_init="0.0" femur_init="1.3" tibia_init="-1.0" />
+	<xacro:leg side="R" position="M" x="0.0" y="-0.100" angle="-${pi/2}" axis="1" coxa_init="0.0" femur_init="1.3" tibia_init="-1.0" />
+	<xacro:leg side="R" position="F" x="0.120" y="-0.060" angle="-${pi/4}" axis="1" coxa_init="0.0" femur_init="1.3" tibia_init="-1.0" />
+	<xacro:leg side="L" position="R" x="-0.120" y="0.060" angle="${pi*3/4}" axis="-1" coxa_init="0.0" femur_init="-1.3" tibia_init="1.0" />
+	<xacro:leg side="L" position="M" x="0.0" y="0.100" angle="${pi/2}" axis="-1" coxa_init="0.0" femur_init="-1.3" tibia_init="1.0" />
+	<xacro:leg side="L" position="F" x="0.120" y="0.060" angle="${pi/4}" axis="-1" coxa_init="0.0" femur_init="-1.3" tibia_init="1.0" />
 </robot>
